Commit message: Working scanning fake controller forced

File: godel/godel_robots/ur/godel_ur10/godel_ur10_support/urdf/swri_demo_cell_macro.xacro (robot description, xacro)
@@ -4,9 +4,9 @@
 <!-- Origin is at the robot (IRB 2400) mounting location -->
 <robot xmlns:xacro="http://ros.org/wiki/xacro">
-  <xacro:property name="demo_cell_width" value="1.8288"/> <!-- 60" table + 12" forward-->
-  <xacro:property name="demo_cell_length" value="1.524"/> <!--36" table + 12" left + 12" right -->
-  <xacro:property name="demo_cell_height" value="2.4384"/> <!--96"  vertical-->
-  <xacro:property name="robot_to_corner_x" value="-0.45"/> <!-- 17.7165" from back -->
-  <xacro:property name="robot_to_corner_y" value="-0.762"/> <!-- middle of width -->
+  <xacro:property name="demo_cell_width" value="2.8288"/> <!-- 60" table + 12" forward-->
+  <xacro:property name="demo_cell_length" value="2.524"/> <!--36" table + 12" left + 12" right -->
+  <xacro:property name="demo_cell_height" value="3.4384"/> <!--96"  vertical-->
+  <xacro:property name="robot_to_corner_x" value="-0.95"/> <!-- 17.7165" from back -->
+  <xacro:property name="robot_to_corner_y" value="-1.262"/> <!-- middle of width -->
   <xacro:property name="demo_cell_wall_thickness" value="0.05"/>
   <!--
@@ -94,5 +94,5 @@
     <parent link="${prefix}demo_cell_corner"/>
     <child link="${prefix}demo_cell_floor"/>
-    <origin xyz="${demo_cell_width / 2.0} ${demo_cell_length / 2.0} ${-0.5 * demo_cell_wall_thickness}"/>
+    <origin xyz="${demo_cell_width / 2.0} ${demo_cell_length / 2.0} ${-0.5 * demo_cell_wall_thickness-0.5}"/>
   </joint>
   </xacro:macro>

Commit message: Blending and edge working

File: godel/godel_robots/ur/godel_ur10/godel_ur10_support/urdf/swri_demo_cell_macro.xacro (robot description, xacro)
@@ -4,9 +4,9 @@
 <!-- Origin is at the robot (IRB 2400) mounting location -->
 <robot xmlns:xacro="http://ros.org/wiki/xacro">
-  <xacro:property name="demo_cell_width" value="2.8288"/> <!-- 60" table + 12" forward-->
-  <xacro:property name="demo_cell_length" value="2.524"/> <!--36" table + 12" left + 12" right -->
-  <xacro:property name="demo_cell_height" value="3.4384"/> <!--96"  vertical-->
-  <xacro:property name="robot_to_corner_x" value="-0.95"/> <!-- 17.7165" from back -->
-  <xacro:property name="robot_to_corner_y" value="-1.262"/> <!-- middle of width -->
+  <xacro:property name="demo_cell_width" value="12.8288"/> <!-- 60" table + 12" forward-->
+  <xacro:property name="demo_cell_length" value="12.524"/> <!--36" table + 12" left + 12" right -->
+  <xacro:property name="demo_cell_height" value="13.4384"/> <!--96"  vertical-->
+  <xacro:property name="robot_to_corner_x" value="-5.95"/> <!-- 17.7165" from back -->
+  <xacro:property name="robot_to_corner_y" value="-6.262"/> <!-- middle of width -->
   <xacro:property name="demo_cell_wall_thickness" value="0.05"/>
   <!--

File: godel/godel_robots/ur/godel_ur10/godel_ur10_support/urdf/ur10_workspace.xacro (robot description, xacro)
@@ -6,5 +6,5 @@
   <link name="world_frame"/>
   <!-- instantiating arm  -->
-  <xacro:ur10_robot prefix="" joint_limited="true"/>
+  <xacro:ur10_robot prefix="" joint_limited="false"/>
   <!-- instantiating end effector  -->
   <xacro:blending_eff_definition prefix=""/>
