Commit message: Changed working env, and fixed simulation

File: godel/godel_robots/ur/godel_ur10/godel_ur10_support/urdf/ur10_workcell.xacro (robot description, xacro)
@@ -28,10 +28,10 @@
   </material>
   <xacro:macro name="swri_demo_cell" params="prefix">
-  <link name="table">
+  <link name="tableTop">
         <visual>
             <geometry>
-                <box size="2.0 0.70 0.860"/>
+                <box size="2.0 0.04 0.860"/>
             </geometry>
-            <origin xyz="0.0 -0.225 0.43" rpy="0 0 0" />
+            <origin xyz="0.0 -0.225 0.76" rpy="0 0 0" />
             <material name="yellow" />
         </visual>
@@ -42,4 +42,13 @@
             <origin xyz="0.0 -0.225 0.44" rpy="0 0 0.0" />
         </collision>
+  </link>
+  <link name="tableBottom">
+        <visual>
+            <geometry>
+                <box size="2.0 0.66 0.860"/>
+            </geometry>
+            <origin xyz="0.0 -0.225 0.41" rpy="0 0 0" />
+            <material name="blue" />
+        </visual>
   </link>
   <link name="back_wall">

File: godel/godel_robots/ur/godel_ur10/godel_ur10_support/urdf/ur10_workspace.xacro (robot description, xacro)
@@ -4,5 +4,5 @@
   <xacro:include filename="$(find ur_description)/urdf/ur10.urdf.xacro"/>
   <material name="blue">
-    <color rgba="0 0 0.8 1"/>
+    <color rgba="0.015 0.341 0.858 1"/>
   </material>
   <material name="white">
@@ -13,5 +13,5 @@
     </material>
   <material name="gray">
-    <color rgba="0.7 0.7 0.7 1"/>
+    <color rgba="0.8 0.8 0.8 1"/>
   </material>
   <material name="yellow">
@@ -21,20 +21,41 @@
     <texture filename="package://godel_ur10_support/urdf/textures/smr-poster.png"/>
   </material>
+  <material name="wood">
+    <texture filename="package://godel_ur10_support/urdf/textures/WoodTexture.jpg"/>
+  </material>
   <link name="world_frame"/>
-  <link name="table">
-        <visual>
-            <geometry>
-                <box size="2.0 0.70 0.860"/>
-            </geometry>
-            <origin xyz="0.0 0.0 0.43" rpy="0 0 0" />
-            <material name="yellow" />
-        </visual>
-        <collision>
-            <geometry>
-                <box size="2.0 0.70 0.860"/>
-            </geometry>
-            <origin xyz="0.0 0.0 0.44" rpy="0 0 0.0" />
-        </collision>
-  </link>
+  <link name="tableTop">
+          <visual>
+              <geometry>
+                  <box size="2.0 0.70 0.04"/>
+              </geometry>
+              <origin xyz="0 0 0.43" rpy="0 0 0" />
+              <material name="wood" />
+          </visual>
+          <collision>
+              <geometry>
+                  <box size="2.0 0.70 0.86"/>
+              </geometry>
+              <origin xyz="0 0 0.03" rpy="0 0 0.0" />
+          </collision>
+    </link>
+    <link name="tableBottom">
+          <visual>
+              <geometry>
+                  <box size="1.96 0.66 0.82"/>
+              </geometry>
+              <origin xyz="0 0 0" rpy="0 0 0" />
+              <material name="blue" />
+          </visual>
+    </link>
+    <link name="robotbase">
+          <visual>
+              <geometry>
+                  <box size="0.18 0.25 0.02"/>
+              </geometry>
+              <origin xyz="0 0 0" rpy="0 0 0" />
+              <material name="gray" />
+          </visual>
+    </link>
     <link name="toolstation">
           <collision>
@@ -85,9 +106,19 @@
     <origin xyz="0.91 0 0.880" rpy="0 0 0"/>
   </joint>
-  <joint name="world_to_table" type="fixed">
-          <parent link="world_frame" />
-          <child link ="table" />
-          <origin xyz="0 0 0" rpy="0 0 0" />
-  </joint>
+    <joint name="world_to_tableBottom" type="fixed">
+            <parent link="world_frame" />
+            <child link ="tableBottom" />
+            <origin xyz="0.0 -0.0 0.41" rpy="0 0 0" />
+    </joint>
+    <joint name="world_to_tableTop" type="fixed">
+            <parent link="world_frame" />
+            <child link ="tableTop" />
+            <origin xyz="0.0 0.0 0.41" rpy="0 0 0" />
+    </joint>
+    <joint name="world_to_robotbase" type="fixed">
+            <parent link="world_frame" />
+            <child link ="robotbase" />
+            <origin xyz="0.91 0 0.87" rpy="0 0 0" />
+    </joint>
   <joint name="world_to_toolstation" type="fixed">
           <parent link="world_frame" />
@@ -103,5 +134,5 @@
           <parent link="back_wall" />
           <child link ="smr-poster" />
-          <origin xyz="0 -0.051 0.30" rpy="0 -1.57 1.57" />
+          <origin xyz="0 -0.055 0.30" rpy="0 -1.57 1.57" />
   </joint>
 </robot>
