Commit message: Working Blending UR10 IRL real robot fake pointcloud glitchy rviz robot flickering to home position

File: godel/godel_robots/ur/godel_ur10/godel_ur10_support/urdf/ur10_workspace.xacro (robot description, xacro)
@@ -3,11 +3,66 @@
   <xacro:include filename="$(find blending_end_effector)/urdf/blending_eff_macro.xacro"/>
   <xacro:include filename="$(find ur_description)/urdf/ur10.urdf.xacro"/>
-  <xacro:include filename="$(find godel_ur10_support)/urdf/swri_demo_cell_macro.xacro"/>
+  <material name="blue">
+    <color rgba="0 0 0.8 1"/>
+  </material>
+  <material name="white">
+    <color rgba="1 1 1 1"/>
+  </material>
+    <material name="black">
+  <color rgba="0.1 0.1 0.1 1"/>
+    </material>
+  <material name="gray">
+    <color rgba="0.7 0.7 0.7 1"/>
+  </material>
+  <material name="yellow">
+    <color rgba="0.9 0.8 0.3 1"/>
+  </material>
+  <material name="poster">
+    <texture filename="package://godel_ur10_support/urdf/textures/poster.png"/>
+  </material>
   <link name="world_frame"/>
+  <link name="table">
+        <visual>
+            <geometry>
+                <box size="2.0 0.70 0.860"/>
+            </geometry>
+            <origin xyz="0.0 0.0 0.43" rpy="0 0 0" />
+            <material name="yellow" />
+        </visual>
+        <collision>
+            <geometry>
+                <box size="2.0 0.70 0.860"/>
+            </geometry>
+            <origin xyz="0.0 0.0 0.44" rpy="0 0 0.0" />
+        </collision>
+  </link>
+  <link name="back_wall">
+        <visual>
+            <geometry>
+                <box size="4.0 0.10 3.0"/>
+            </geometry>
+            <origin xyz="0 0 0" rpy="0 0 0" />
+            <material name="gray" />
+        </visual>
+        <collision>
+            <geometry>
+                <box size="4.0 0.10 3.0"/>
+            </geometry>
+            <origin xyz="0 0 0" rpy="0 0 0" />
+        </collision>
+  </link>
+  <link name="poster">
+          <visual>
+              <geometry>
+                  <box size="1.5 1.059 0.0"/>
+              </geometry>
+               <origin xyz="0 0 0" rpy="0 0 0" />
+              <material name="poster" />
+          </visual>
+  </link>
   <!-- instantiating arm  -->
   <xacro:ur10_robot prefix="" joint_limited="false"/>
   <!-- instantiating end effector  -->
   <xacro:blending_eff_definition prefix=""/>
-  <xacro:swri_demo_cell prefix=""/>
   <!-- Attach the end effector to the end of the robot arm (tool0) -->
   <joint name="link_t_to_eff" type="fixed">
@@ -20,10 +75,20 @@
     <parent link="world_frame"/>
     <child link="base_link"/>
-    <origin xyz="0 0 0" rpy="0 0 0"/>
+    <origin xyz="0.91 0 0.880" rpy="0 0 0"/>
   </joint>
-  <joint name="world_to_demo_cell" type="fixed">
-    <parent link="world_frame"/>
-    <child link="demo_cell_base_link"/>
-    <origin xyz="0 0 0" rpy="0 0 0"/>
+  <joint name="world_to_table" type="fixed">
+          <parent link="world_frame" />
+          <child link ="table" />
+          <origin xyz="0 0 0" rpy="0 0 0" />
+  </joint>
+  <joint name="world_to_back_wall" type="fixed">
+          <parent link="world_frame" />
+          <child link ="back_wall" />
+          <origin xyz="0.0 0.40 1.5" rpy="0 0 0" />
+  </joint>
+  <joint name="world_to_poster" type="fixed">
+          <parent link="back_wall" />
+          <child link ="poster" />
+          <origin xyz="0 -0.051 0.30" rpy="0 -1.57 1.57" />
   </joint>
 </robot>

Commit message: Added camera box above table, moved depth frame

File: godel/godel_robots/ur/godel_ur10/godel_ur10_support/urdf/ur10_workspace.xacro (robot description, xacro)
@@ -52,4 +52,19 @@
         </collision>
   </link>
+  <link name="camera">
+          <visual>
+              <geometry>
+                  <box size="0.50 0.35 0.35"/>
+              </geometry>
+              <origin xyz="0 0 0" rpy="0 0 0" />
+              <material name="yellow" />
+          </visual>
+          <collision>
+              <geometry>
+                  <box size="0.50 0.35 0.35"/>
+              </geometry>
+              <origin xyz="0 0 0" rpy="0 0 0" />
+          </collision>
+  </link>
   <link name="poster">
           <visual>
@@ -82,4 +97,9 @@
           <origin xyz="0 0 0" rpy="0 0 0" />
   </joint>
+  <joint name="world_to_camera" type="fixed">
+          <parent link="world_frame" />
+          <child link ="camera" />
+          <origin xyz="0.10 0 2.28" rpy="0 0 0" />
+  </joint>
   <joint name="world_to_back_wall" type="fixed">
           <parent link="world_frame" />

Commit message: Update

File: godel/godel_robots/ur/godel_ur10/godel_ur10_support/urdf/ur10_workspace.xacro (robot description, xacro)
@@ -59,10 +59,10 @@
     </link>
     <link name="toolstation">
-          <collision>
-              <geometry>
-                  <box size="1.0 0.10 2.0"/>
-              </geometry>
-              <origin xyz="0.0 0.0 0.0" rpy="0 0 0.0" />
-          </collision>
+          <visual>
+            <geometry>
+                <mesh filename="package://godel_ur10_support/meshes/grinder_system.stl"/>
+            </geometry>
+            <origin xyz="0.0 -1.4 0.0" rpy="0 0 1.57" />
+          </visual>
     </link>
   <link name="back_wall">
@@ -139,5 +139,5 @@
           <parent link="world_frame" />
           <child link ="toolstation" />
-          <origin xyz="0.5 -1.0 1.0" rpy="0 0 0" />
+          <origin xyz="0.0 0.0 0.0" rpy="0 0 0.0" />
   </joint>
   <joint name="world_to_back_wall" type="fixed">

Commit message: Might all be working, did the first small grind already

File: godel/godel_robots/ur/godel_ur10/godel_ur10_support/urdf/ur10_workspace.xacro (robot description, xacro)
@@ -58,5 +58,5 @@
           </visual>
     </link>
-    <link name="toolstation">
+    <link name="toolstation_side">
           <visual>
             <geometry>
@@ -136,7 +136,7 @@
             <origin xyz="0.91 0 0.87" rpy="0 0 0" />
     </joint>
-  <joint name="world_to_toolstation" type="fixed">
+  <joint name="world_to_toolstation_side" type="fixed">
           <parent link="world_frame" />
-          <child link ="toolstation" />
+          <child link ="toolstation_side" />
           <origin xyz="0.0 0.0 0.0" rpy="0 0 0.0" />
   </joint>

Commit message: Small changes in the working env, and added the motordriver arduino rosserial to the launchfile

File: godel/godel_robots/ur/godel_ur10/godel_ur10_support/urdf/ur10_workspace.xacro (robot description, xacro)
@@ -61,8 +61,15 @@
           <visual>
             <geometry>
-                <mesh filename="package://godel_ur10_support/meshes/grinder_system.stl"/>
+                <mesh filename="package://godel_ur10_support/meshes/grinder_system_small.stl"/>
             </geometry>
-            <origin xyz="0.0 -1.4 0.0" rpy="0 0 1.57" />
+            <origin xyz="0.0 0.0 0.0" rpy="0 0 0" />
+            <material name="gray" />
           </visual>
+          <collision>
+              <geometry>
+                  <mesh filename="package://godel_ur10_support/meshes/grinder_system_small.stl"/>
+              </geometry>
+              <origin xyz="0.0 0.0 0.0" rpy="0 0 0" />
+          </collision>
     </link>
   <link name="back_wall">
@@ -82,11 +89,4 @@
   </link>
   <link name="side_wall">
-        <visual>
-            <geometry>
-                <box size="0.10 1.0 3.0"/>
-            </geometry>
-            <origin xyz="0 0 0" rpy="0 0 0" />
-            <material name="gray" />
-        </visual>
         <collision>
             <geometry>
@@ -139,5 +139,5 @@
           <parent link="world_frame" />
           <child link ="toolstation_side" />
-          <origin xyz="0.0 0.0 0.0" rpy="0 0 0.0" />
+          <origin xyz="0.945 -0.35 0.80" rpy="0 0 -1.57" />
   </joint>
   <joint name="world_to_back_wall" type="fixed">
