Commit message: scanNplan launches with ur_10

File: godel/godel_robots/blending_end_effector/urdf/blending_eff_macro.xacro (robot description, xacro)
@@ -22,6 +22,6 @@
   <xacro:macro name="blending_eff_definition" params="prefix">
     <!-- eff_frame is Base Link -->
-    <link name="${prefix}eff_frame"/>
-    <link name="${prefix}adapter_tube">
+    <link name="eff_frame"/>
+    <link name="adapter_tube">
       <visual>
         <geometry>
@@ -38,10 +38,10 @@
       </collision>
     </link>
-    <joint name="${prefix}eff_frame_to_adapter_tube" type="fixed">
-        <parent link="${prefix}eff_frame"/>
-        <child link="${prefix}adapter_tube"/>
+    <joint name="eff_frame_to_adapter_tube" type="fixed">
+        <parent link="eff_frame"/>
+        <child link="adapter_tube"/>
         <origin xyz="0 0 0" rpy="0 0 0"/>
     </joint>
-    <link name="${prefix}bracket">
+    <link name="bracket">
       <visual>
         <geometry>
@@ -58,10 +58,10 @@
       </collision>
     </link>
-    <joint name="${prefix}adapter_tube_to_bracket" type="fixed">
-      <parent link="${prefix}adapter_tube"/>
-      <child link="${prefix}bracket"/>
+    <joint name="adapter_tube_to_bracket" type="fixed">
+      <parent link="adapter_tube"/>
+      <child link="bracket"/>
       <origin xyz="0 0 0" rpy="0 0 0"/>
     </joint>
-    <link name="${prefix}blending_tool">
+    <link name="blending_tool">
         <visual>
             <geometry>
@@ -73,9 +73,9 @@
         </visual>
     </link>
-    <joint name="${prefix}bracket_to_blending_tool" type="fixed">
-        <parent link="${prefix}bracket"/>
-        <child link="${prefix}blending_tool"/>
+    <joint name="bracket_to_blending_tool" type="fixed">
+        <parent link="bracket"/>
+        <child link="blending_tool"/>
     </joint>
-    <link name="${prefix}ensenso">
+    <link name="ensenso">
         <visual>
             <geometry>
@@ -87,9 +87,9 @@
         </visual>
     </link>
-    <joint name="${prefix}bracket_to_ensenso" type="fixed">
-        <parent link="${prefix}bracket"/>
-        <child link="${prefix}ensenso"/>
+    <joint name="bracket_to_ensenso" type="fixed">
+        <parent link="bracket"/>
+        <child link="ensenso"/>
     </joint>
-    <link name="${prefix}keyence">
+    <link name="keyence">
         <visual>
             <geometry>
@@ -101,45 +101,45 @@
         </visual>
     </link>
-    <joint name="${prefix}bracket_to_keyence" type="fixed">
-        <parent link="${prefix}bracket"/>
-        <child link="${prefix}keyence"/>
+    <joint name="bracket_to_keyence" type="fixed">
+        <parent link="bracket"/>
+        <child link="keyence"/>
     </joint>
     <!-- Frames for the motorized spindle on the end-->
-    <link name="${prefix}chuck_tip_frame"/> <!--The tip of the chuck-->
-    <link name="${prefix}tcp_frame"/> <!--The actual 'useful' work frame-->
-    <joint name="${prefix}bracket_to_chuck" type="fixed">
-        <parent link="${prefix}bracket"/>
-        <child link="${prefix}chuck_tip_frame"/>
+    <link name="chuck_tip_frame"/> <!--The tip of the chuck-->
+    <link name="tcp_frame"/> <!--The actual 'useful' work frame-->
+    <joint name="bracket_to_chuck" type="fixed">
+        <parent link="bracket"/>
+        <child link="chuck_tip_frame"/>
         <origin xyz="${chuck_tcp_x} ${chuck_tcp_y} ${chuck_tcp_z}" rpy="0 -${half_pi} 0"/>
     </joint>
-    <joint name="${prefix}chuck_to_blend_tcp_frame" type="fixed">
-        <parent link="${prefix}chuck_tip_frame"/>
-        <child link="${prefix}tcp_frame"/>
+    <joint name="chuck_to_blend_tcp_frame" type="fixed">
+        <parent link="chuck_tip_frame"/>
+        <child link="tcp_frame"/>
         <origin xyz="${blend_tcp_x} ${blend_tcp_y} ${blend_tcp_z}" rpy="0 0 0"/>
     </joint>
     <!--Frames for the keyence profilometer-->
-    <link name="${prefix}keyence_sensor_optical_frame"/>  <!--The emitter lens-->
-    <link name="${prefix}keyence_tcp_frame"/> <!--The nominal scan location (8cm forward of emitter)-->
-    <joint name="${prefix}bracket_to_keyence_sof" type="fixed">
-        <parent link="${prefix}bracket"/>
-        <child link="${prefix}keyence_sensor_optical_frame"/>
+    <link name="keyence_sensor_optical_frame"/>  <!--The emitter lens-->
+    <link name="keyence_tcp_frame"/> <!--The nominal scan location (8cm forward of emitter)-->
+    <joint name="bracket_to_keyence_sof" type="fixed">
+        <parent link="bracket"/>
+        <child link="keyence_sensor_optical_frame"/>
         <origin xyz="${keyence_tcp_x} ${keyence_tcp_y} ${keyence_tcp_z}" rpy="${half_pi} ${half_pi} 0 "/>
     </joint>
-    <joint name="${prefix}bracket_to_keyence_tcp_f" type="fixed">
-        <parent link="${prefix}bracket"/>
-        <child link="${prefix}keyence_tcp_frame"/>
+    <joint name="bracket_to_keyence_tcp_f" type="fixed">
+        <parent link="bracket"/>
+        <child link="keyence_tcp_frame"/>
         <origin xyz="${keyence_tcp_x} ${keyence_tcp_y} ${keyence_tcp_z}" rpy="-${half_pi} ${half_pi} 0"/>
     </joint>
     <!--Frames related to the motion of the camera-->
-    <link name="${prefix}ensenso_sensor_optical_frame"/>
-    <link name="${prefix}kinect2_move_frame"/>
-    <joint name="${prefix}bracket_to_ensenso_sof" type="fixed">
-        <parent link="${prefix}bracket"/>
-        <child link="${prefix}ensenso_sensor_optical_frame"/>
+    <link name="ensenso_sensor_optical_frame"/>
+    <link name="kinect2_move_frame"/>
+    <joint name="bracket_to_ensenso_sof" type="fixed">
+        <parent link="bracket"/>
+        <child link="ensenso_sensor_optical_frame"/>
         <origin xyz="${ensenso_optical_x} ${ensenso_optical_y} ${ensenso_optical_z}" rpy="0 0 0"/>
     </joint>
-    <joint name="${prefix}ensenso_move_frame_join" type="fixed">
-      <parent link="${prefix}ensenso_sensor_optical_frame"/>
-      <child link="${prefix}kinect2_move_frame"/>
+    <joint name="ensenso_move_frame_join" type="fixed">
+      <parent link="ensenso_sensor_optical_frame"/>
+      <child link="kinect2_move_frame"/>
       <origin rpy="0 -${half_pi} 0"/>
     </joint>

Commit message: Camera on robot arm

File: godel/godel_robots/blending_end_effector/urdf/blending_eff_macro.xacro (robot description, xacro)
@@ -13,28 +13,41 @@
   <xacro:property name="kinect_mount_y" value="-0.065"/>
   <xacro:property name="kinect_mount_z" value="0.15"/>
-  <xacro:property name="blend_tcp_x" value="0"/>
+  <xacro:property name="blend_tcp_x" value="0.040"/>
   <xacro:property name="blend_tcp_y" value="0"/>
-  <xacro:property name="blend_tcp_z" value="0.040"/> <!-- TBD -->
-  <xacro:property name="chuck_tcp_x" value="-0.2507"/>
-  <xacro:property name="chuck_tcp_y" value="-0.0035"/>
-  <xacro:property name="chuck_tcp_z" value="0.1228"/>
+  <xacro:property name="blend_tcp_z" value="0.0"/> <!-- TBD -->
+  <xacro:property name="chuck_tcp_x" value="0.0"/>
+  <xacro:property name="chuck_tcp_y" value="0.0"/>
+  <xacro:property name="chuck_tcp_z" value="0.15"/>
   <xacro:property name="half_pi" value="1.5707963267948966"/>
   <xacro:macro name="blending_eff_definition" params="prefix">
     <!-- eff_frame is Base Link -->
     <link name="eff_frame"/>
+    <link name="UR10_EOAT_rotate"/>
+    <link name="UR10_EOAT">
+        <visual>
+            <geometry>
+              <mesh filename="package://blending_end_effector/meshes/visual/UR10_EOAT.stl"/>
+            </geometry>
+            <material name="grey">
+              <color rgba="0.5 0.5 0.5 1.0"/>
+            </material>
+        </visual>
+        <collision>
+            <geometry>
+              <mesh filename="package://blending_end_effector/meshes/collision/UR10_EOAT_Collision.stl"/>
+            </geometry>
+        </collision>
+    </link>
+    <joint name="eff_frame_to_UR10_EOAT_rotate" type="fixed">
+        <parent link="eff_frame"/>
+        <child link="UR10_EOAT_rotate"/>
+        <origin xyz="0 0 0" rpy="0 0 0.785"/>
+    </joint>
+    <joint name="UR10_EOAT_rotate_to_UR10_EOAT" type="fixed">
+        <parent link="UR10_EOAT_rotate"/>
+        <child link="UR10_EOAT"/>
+        <origin xyz="0 0.08 0" rpy="0 0 0"/>
+    </joint>
     <link name="adapter_tube">
-      <visual>
-        <geometry>
-          <mesh filename="package://blending_end_effector/meshes/visual/Adapter_Tube.STL"/>
-        </geometry>
-        <material name="grey">
-          <color rgba="0.5 0.5 0.5 1.0"/>
-        </material>
-      </visual>
-      <collision>
-        <geometry>
-          <mesh filename="package://blending_end_effector/meshes/collision/adapter_tube_convex_hull.STL"/>
-        </geometry>
-      </collision>
     </link>
     <joint name="eff_frame_to_adapter_tube" type="fixed">
@@ -44,17 +57,4 @@
     </joint>
     <link name="bracket">
-      <visual>
-        <geometry>
-          <mesh filename="package://blending_end_effector/meshes/visual/Tool_Mounting_Plate.STL"/>
-        </geometry>
-        <material name="grey">
-          <color rgba="0.5 0.5 0.5 1.0"/>
-        </material>
-      </visual>
-      <collision>
-        <geometry>
-          <mesh filename="package://blending_end_effector/meshes/collision/EE_and_Tool_Changer_convex_hull.STL"/>
-        </geometry>
-      </collision>
     </link>
     <joint name="adapter_tube_to_bracket" type="fixed">
@@ -64,12 +64,4 @@
     </joint>
     <link name="blending_tool">
-        <visual>
-            <geometry>
-                <mesh filename="package://blending_end_effector/meshes/visual/Blending_Tool.STL"/>
-            </geometry>
-            <material name="red">
-                <color rgba="1 0 0 1"/>
-            </material>
-        </visual>
     </link>
     <joint name="bracket_to_blending_tool" type="fixed">
@@ -78,12 +70,4 @@
     </joint>
     <link name="ensenso">
-        <visual>
-            <geometry>
-                <mesh filename="package://blending_end_effector/meshes/visual/Ensenso.STL"/>
-            </geometry>
-            <material name="blue">
-                <color rgba="0 0 1 1"/>
-            </material>
-        </visual>
     </link>
     <joint name="bracket_to_ensenso" type="fixed">
@@ -92,12 +76,4 @@
     </joint>
     <link name="keyence">
-        <visual>
-            <geometry>
-                <mesh filename="package://blending_end_effector/meshes/visual/Laser_Sensor.STL"/>
-            </geometry>
-            <material name="yellow">
-                <color rgba="1 1 0 1"/>
-            </material>
-        </visual>
     </link>
     <joint name="bracket_to_keyence" type="fixed">

File: godel/godel_robots/ur/godel_ur10/godel_ur10_support/urdf/ur10_workcell.xacro (robot description, xacro)
@@ -24,6 +24,6 @@
     <color rgba="0.9 0.8 0.3 1"/>
   </material>
-  <material name="poster">
-              <texture filename="package://godel_ur10_support/urdf/textures/poster.png"/>
+  <material name="smr-poster">
+              <texture filename="package://godel_ur10_support/urdf/textures/smr-poster.png"/>
   </material>
   <xacro:macro name="swri_demo_cell" params="prefix">
@@ -58,5 +58,5 @@
         </collision>
   </link>
-  <link name="poster">
+  <link name="smr-poster">
           <visual>
               <geometry>
@@ -64,5 +64,5 @@
               </geometry>
                <origin xyz="2.0 0.0 -0.675" rpy="0 0 0" />
-              <material name="poster" />
+              <material name="smr-poster" />
           </visual>
   </link>
@@ -82,7 +82,7 @@
         <origin xyz="0 0 0" rpy="0 0 0" />
   </joint>
-  <joint name="world_to_poster" type="fixed">
+  <joint name="world_to_smr-poster" type="fixed">
         <parent link="${prefix}demo_cell_base_link" />
-        <child link ="poster" />
+        <child link ="smr-poster" />
         <origin xyz="0 0 0" rpy="0 -1.57 1.57" />
   </joint>

File: godel/godel_robots/ur/godel_ur10/godel_ur10_support/urdf/ur10_workspace.xacro (robot description, xacro)
@@ -18,6 +18,6 @@
     <color rgba="0.9 0.8 0.3 1"/>
   </material>
-  <material name="poster">
-    <texture filename="package://godel_ur10_support/urdf/textures/poster.png"/>
+  <material name="smr-poster">
+    <texture filename="package://godel_ur10_support/urdf/textures/smr-poster.png"/>
   </material>
   <link name="world_frame"/>
@@ -52,20 +52,5 @@
         </collision>
   </link>
-  <link name="camera">
-          <visual>
-              <geometry>
-                  <box size="0.50 0.35 0.35"/>
-              </geometry>
-              <origin xyz="0 0 0" rpy="0 0 0" />
-              <material name="yellow" />
-          </visual>
-          <collision>
-              <geometry>
-                  <box size="0.50 0.35 0.35"/>
-              </geometry>
-              <origin xyz="0 0 0" rpy="0 0 0" />
-          </collision>
-  </link>
-  <link name="poster">
+  <link name="smr-poster">
           <visual>
               <geometry>
@@ -73,5 +58,5 @@
               </geometry>
                <origin xyz="0 0 0" rpy="0 0 0" />
-              <material name="poster" />
+              <material name="smr-poster" />
           </visual>
   </link>
@@ -97,9 +82,4 @@
           <origin xyz="0 0 0" rpy="0 0 0" />
   </joint>
-  <joint name="world_to_camera" type="fixed">
-          <parent link="world_frame" />
-          <child link ="camera" />
-          <origin xyz="0.10 0 2.28" rpy="0 0 0" />
-  </joint>
   <joint name="world_to_back_wall" type="fixed">
           <parent link="world_frame" />
@@ -107,7 +87,7 @@
           <origin xyz="0.0 0.40 1.5" rpy="0 0 0" />
   </joint>
-  <joint name="world_to_poster" type="fixed">
+  <joint name="world_to_smr-poster" type="fixed">
           <parent link="back_wall" />
-          <child link ="poster" />
+          <child link ="smr-poster" />
           <origin xyz="0 -0.051 0.30" rpy="0 -1.57 1.57" />
   </joint>

Commit message: Camera Frame and tool frame in correct position

File: godel/godel_robots/blending_end_effector/urdf/blending_eff_macro.xacro (robot description, xacro)
@@ -13,7 +13,7 @@
   <xacro:property name="kinect_mount_y" value="-0.065"/>
   <xacro:property name="kinect_mount_z" value="0.15"/>
-  <xacro:property name="blend_tcp_x" value="0.040"/>
-  <xacro:property name="blend_tcp_y" value="0"/>
-  <xacro:property name="blend_tcp_z" value="0.0"/> <!-- TBD -->
+  <xacro:property name="blend_tcp_x" value="0.0"/>
+  <xacro:property name="blend_tcp_y" value="0.0"/>
+  <xacro:property name="blend_tcp_z" value="0.04"/> <!-- TBD -->
   <xacro:property name="chuck_tcp_x" value="0.0"/>
   <xacro:property name="chuck_tcp_y" value="0.0"/>
@@ -87,5 +87,5 @@
         <parent link="bracket"/>
         <child link="chuck_tip_frame"/>
-        <origin xyz="${chuck_tcp_x} ${chuck_tcp_y} ${chuck_tcp_z}" rpy="0 -${half_pi} 0"/>
+        <origin xyz="${chuck_tcp_x} ${chuck_tcp_y} ${chuck_tcp_z}" rpy="0 0 0.78"/>
     </joint>
     <joint name="chuck_to_blend_tcp_frame" type="fixed">

File: godel/godel_robots/ur/godel_ur10/godel_ur10_support/urdf/ur10_workspace.xacro (robot description, xacro)
@@ -37,4 +37,12 @@
         </collision>
   </link>
+    <link name="toolstation">
+          <collision>
+              <geometry>
+                  <box size="1.0 0.10 2.0"/>
+              </geometry>
+              <origin xyz="0.0 0.0 0.0" rpy="0 0 0.0" />
+          </collision>
+    </link>
   <link name="back_wall">
         <visual>
@@ -82,4 +90,9 @@
           <origin xyz="0 0 0" rpy="0 0 0" />
   </joint>
+  <joint name="world_to_toolstation" type="fixed">
+          <parent link="world_frame" />
+          <child link ="toolstation" />
+          <origin xyz="0.5 -1.0 1.0" rpy="0 0 0" />
+  </joint>
   <joint name="world_to_back_wall" type="fixed">
           <parent link="world_frame" />

Commit message: Fixed USB grinder arduino problem on laptop Matthijs, to make it work on other laptop add /grinder_switch_arduino remap to udef rules

File: godel/godel_robots/blending_end_effector/urdf/blending_eff_macro.xacro (robot description, xacro)
@@ -14,5 +14,5 @@
   <xacro:property name="kinect_mount_z" value="0.15"/>
   <xacro:property name="blend_tcp_x" value="0.0"/>
-  <xacro:property name="blend_tcp_y" value="0.0"/>
+  <xacro:property name="blend_tcp_y" value="-0.05"/>
   <xacro:property name="blend_tcp_z" value="0.04"/> <!-- TBD -->
   <xacro:property name="chuck_tcp_x" value="0.0"/>
@@ -92,5 +92,5 @@
         <parent link="chuck_tip_frame"/>
         <child link="tcp_frame"/>
-        <origin xyz="${blend_tcp_x} ${blend_tcp_y} ${blend_tcp_z}" rpy="0 0 0"/>
+        <origin xyz="${blend_tcp_x} ${blend_tcp_y} ${blend_tcp_z}" rpy="0.1745 0 0"/>
     </joint>
     <!--Frames for the keyence profilometer-->

File: godel/godel_robots/ur/godel_ur10/godel_ur10_support/urdf/ur10_workspace.xacro (robot description, xacro)
@@ -81,4 +81,19 @@
         </collision>
   </link>
+  <link name="side_wall">
+        <visual>
+            <geometry>
+                <box size="0.10 1.0 3.0"/>
+            </geometry>
+            <origin xyz="0 0 0" rpy="0 0 0" />
+            <material name="gray" />
+        </visual>
+        <collision>
+            <geometry>
+                <box size="0.1 1.0 3.0"/>
+            </geometry>
+            <origin xyz="0 0 0" rpy="0 0 0" />
+        </collision>
+  </link>
   <link name="smr-poster">
           <visual>
@@ -131,4 +146,9 @@
           <origin xyz="0.0 0.40 1.5" rpy="0 0 0" />
   </joint>
+  <joint name="world_to_side_wall" type="fixed">
+          <parent link="world_frame" />
+          <child link ="side_wall" />
+          <origin xyz="1.70 -0.15 1.5" rpy="0 0 0" />
+  </joint>
   <joint name="world_to_smr-poster" type="fixed">
           <parent link="back_wall" />

Commit message: Fixed real pointcloud

File: godel/godel_robots/blending_end_effector/urdf/blending_eff_macro.xacro (robot description, xacro)
@@ -110,4 +110,6 @@
     <link name="ensenso_sensor_optical_frame"/>
     <link name="kinect2_move_frame"/>
+    <link name="kinect2_between_move_frame"/>
+    <link name="kinect2_link_move_frame"/>
     <joint name="bracket_to_ensenso_sof" type="fixed">
         <parent link="bracket"/>
@@ -120,4 +122,14 @@
       <origin rpy="0 -${half_pi} 0"/>
     </joint>
+    <joint name="kinect_link_between_move_frame_join" type="fixed">
+              <parent link="kinect2_move_frame"/>
+              <child link="kinect2_between_move_frame"/>
+              <origin xyz="-0.08 0.08 0.228" rpy="2.35619 0 0"/>
+        </joint>
+    <joint name="kinect_link_move_frame_join" type="fixed">
+          <parent link="kinect2_between_move_frame"/>
+          <child link="kinect2_link_move_frame"/>
+          <origin xyz="0 0 0" rpy="0 0 1.570796"/>
+    </joint>
   </xacro:macro>
 </robot>
